File: xt-cf-mini.kicad_pcb (KiCad board)
At the start: 2 copper layers, 81.3 x 49 mm, 32 parts, among them P1 CF_CARD, P2 LED, SW1 ROM Enable, SW2 ROM Write Enable, SW3 ROM Addr, SW4 IDE Addr, U1 28C64, U2 74LS688, U3 74LS688, U4 74LS32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

Commit message: Add files via upload
Routing:
- net GND: track 198.7 -> 192.9 mm
- net VCC: track 308.5 -> 311.3 mm
- net /~CF_CS1: track 40.4 -> 42.2 mm
- net /D6: track 79.5 -> 81.2 mm
- net /~ROMW: track 93.1 -> 94.7 mm
- net /D7: track 84.5 -> 86.0 mm
- net /~CF_CS0: track 31.5 -> 32.8 mm
- net Net-(RN1-Pad3): track 24.7 -> 25.9 mm
- net Net-(RN3-Pad3): track 71.0 -> 72.2 mm
- net Net-(D1-Pad2): track 39.4 -> 40.5 mm
- net Net-(RN3-Pad1): track 61.7 -> 62.8 mm
- net /AEN: track 92.7 -> 93.6 mm
- net /~MEMW: track 119.3 -> 120.2 mm
- net /A12: track 58.8 -> 59.7 mm
- net Net-(RN2-Pad2): track 50.6 -> 49.8 mm
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Other:
- board text removed: "Do not populate"
- board text removed: "THIS END TO PC REAR"

Commit message: Add files via upload
Other:
- board text added: "= Default"
Changed lines of the file:
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@@
   (general
     (thickness 1.6002)
-    (drawings 63)
+    (drawings 68)
     (tracks 1179)
     (zones 0)
@@
       (xy 0.500964 3.601424)) (layer B.SilkS) (width 0.01))
   )
+  (gr_line (start 121.796 120.6025) (end 121.796 117.3005) (layer B.SilkS) (width 0.1524))
+  (gr_line (start 135.639 117.3005) (end 135.639 124.6665) (layer B.SilkS) (width 0.1524))
+  (gr_line (start 135.639 105.7275) (end 121.796 105.7275) (layer B.SilkS) (width 0.1524))
+  (gr_circle (center 118.9355 110.0455) (end 118.9355 109.7915) (layer B.SilkS) (width 0.5))
+  (gr_text "= Default" (at 118.872 114.427 90) (layer B.SilkS)
+    (effects (font (size 0.9 0.9) (thickness 0.1524)) (justify mirror))
+  )
+  (gr_circle (center 130.2385 125.349) (end 130.4925 125.349) (layer B.SilkS) (width 0.5))
+  (gr_circle (center 124.206 114.3635) (end 124.46 114.3635) (layer B.SilkS) (width 0.5))
   (gr_text "THIS END" (at 172.593 93.218) (layer B.SilkS)
     (effects (font (size 2.032 1.524) (thickness 0.3048)) (justify mirror))
@@
     (effects (font (size 1.5 1.2) (thickness 0.2)) (justify left mirror))
   )
-  (gr_line (start 133.7975 115.6495) (end 119.9545 115.6495) (layer B.SilkS) (width 0.1524))
-  (gr_line (start 119.9545 112.0935) (end 133.7975 112.0935) (layer B.SilkS) (width 0.1524))
-  (gr_line (start 119.9545 112.0935) (end 119.9545 109.0455) (layer B.SilkS) (width 0.1524))
-  (gr_line (start 133.7975 109.0455) (end 133.7975 115.2685) (layer B.SilkS) (width 0.1524))
-  (gr_line (start 119.9545 109.0455) (end 133.7975 109.0455) (layer B.SilkS) (width 0.1524))
-  (gr_line (start 133.7975 115.2685) (end 121.6055 115.2685) (layer B.SilkS) (width 0.1524))
-  (gr_line (start 121.6055 109.0455) (end 121.6055 115.2685) (layer B.SilkS) (width 0.1524))
-  (gr_line (start 121.6055 117.3005) (end 121.6055 124.6665) (layer B.SilkS) (width 0.1524))
-  (gr_line (start 119.9545 120.6025) (end 133.7975 120.6025) (layer B.SilkS) (width 0.1524))
-  (gr_line (start 119.9545 120.6025) (end 119.9545 117.3005) (layer B.SilkS) (width 0.1524))
-  (gr_line (start 133.7975 124.6665) (end 121.6055 124.6665) (layer B.SilkS) (width 0.1524))
-  (gr_line (start 133.7975 117.3005) (end 133.7975 124.6665) (layer B.SilkS) (width 0.1524))
-  (gr_line (start 119.9545 117.3005) (end 133.7975 117.3005) (layer B.SilkS) (width 0.1524))
+  (gr_line (start 135.639 115.6495) (end 121.796 115.6495) (layer B.SilkS) (width 0.1524))
+  (gr_line (start 121.796 110.506) (end 135.639 110.506) (layer B.SilkS) (width 0.1524))
+  (gr_line (start 121.796 110.506) (end 121.796 107.458) (layer B.SilkS) (width 0.1524))
+  (gr_line (start 135.639 107.458) (end 135.639 113.681) (layer B.SilkS) (width 0.1524))
+  (gr_line (start 121.796 107.458) (end 135.639 107.458) (layer B.SilkS) (width 0.1524))
+  (gr_line (start 135.639 113.681) (end 123.447 113.681) (layer B.SilkS) (width 0.1524))
+  (gr_line (start 123.447 107.458) (end 123.447 113.681) (layer B.SilkS) (width 0.1524))
+  (gr_line (start 123.447 117.3005) (end 123.447 124.6665) (layer B.SilkS) (width 0.1524))
+  (gr_line (start 121.796 120.6025) (end 135.639 120.6025) (layer B.SilkS) (width 0.1524))
+  (gr_line (start 135.639 124.6665) (end 123.447 124.6665) (layer B.SilkS) (width 0.1524))
+  (gr_line (start 121.796 117.3005) (end 135.639 117.3005) (layer B.SilkS) (width 0.1524))
   (gr_line (start 105.8545 125.349) (end 101.981 125.349) (layer B.SilkS) (width 0.1524))
   (gr_line (start 105.791 106.045) (end 101.981 106.045) (layer B.SilkS) (width 0.1524))
@@
     (effects (font (size 1 1) (thickness 0.2)) (justify mirror))
   )
-  (gr_text "IDE I/O Addr." (at 134.0515 108.2835) (layer B.SilkS)
+  (gr_text "IDE I/O Addr." (at 135.5725 106.696) (layer B.SilkS)
     (effects (font (size 0.9 0.9) (thickness 0.1524)) (justify left mirror))
   )
-  (gr_text "Boot ROM I/O Addr." (at 134.0515 116.5385) (layer B.SilkS)
+  (gr_text "Boot ROM I/O Addr." (at 135.509 116.586) (layer B.SilkS)
     (effects (font (size 0.9 0.9) (thickness 0.1524)) (justify left mirror))
   )
@@
     (effects (font (size 1.5 1.5) (thickness 0.3)) (justify mirror))
   )
-  (gr_text "123\n111 C000\n110 C400\n101 C800\n100 CC00\n011 D000\n010 D400\n001 D800\n000 DC00" (at 126.9395 117.5545 90) (layer B.SilkS)
+  (gr_text "123\n111 C000\n110 C400\n101 C800\n100 CC00\n011 D000\n010 D400\n001 D800\n000 DC00" (at 128.781 117.5545 90) (layer B.SilkS)
     (effects (font (size 0.9 0.9) (thickness 0.1524)) (justify left mirror))
   )
-  (gr_text "123\n111 300\n110 320\n101 340\n100 360\n011 380\n010 3A0\n001 3C0\n000 3E0" (at 126.9395 109.1725 90) (layer B.SilkS)
+  (gr_text "123\n111 300\n110 320\n101 340\n100 360\n011 380\n010 3A0\n001 3C0\n000 3E0" (at 128.781 107.585 90) (layer B.SilkS)
     (effects (font (size 0.9 0.9) (thickness 0.1524)) (justify left mirror))
   )

Commit message: Add files via upload
Routing:
- net GND: track 192.9 -> 198.6 mm
- net VCC: track 311.3 -> 307.4 mm
- net Net-(RN2-Pad2): track 49.8 -> 48.8 mm
- net Net-(RN1-Pad1): track 16.0 -> 15.0 mm
- net Net-(JP1-Pad2): track 65.4 -> 64.7 mm

Commit message: Add files via upload
Parts:
- moved D1 2.55 mm to (110.5, 100.4), turned to 180 degrees
Connections:
- RN4 pad 1: Net-(D1-Pad1) -> Net-(D1-Pad2)
- U5 pad 10: Net-(D1-Pad2) -> Net-(D1-Pad1)
Routing:
- net Net-(D1-Pad2): track 40.5 -> 11.7 mm, vias 1 -> 0
- net Net-(D1-Pad1): track 11.7 -> 40.5 mm, vias 0 -> 1
Changed lines of the file:
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@@
-(kicad_pcb (version 20171130) (host pcbnew "(5.0.0)")
+(kicad_pcb (version 20171130) (host pcbnew "(5.0.1)-3")
   (general
     (thickness 1.6002)
-    (drawings 68)
+    (drawings 70)
     (tracks 1099)
     (zones 0)
@@
     (pad_drill 0.8128)
     (pad_to_mask_clearance 0.254)
+    (solder_mask_min_width 0.25)
     (aux_axis_origin 0 0)
     (visible_elements 7FFFFFFF)
@@
       (net 52 "Net-(U5-Pad11)"))
     (pad 10 smd rect (at 2.7 -1.27) (size 1.5 0.6) (layers Back B.Paste B.Mask)
-      (net 46 "Net-(D1-Pad2)"))
+      (net 47 "Net-(D1-Pad1)"))
     (pad 9 smd rect (at 2.7 -2.54) (size 1.5 0.6) (layers Back B.Paste B.Mask)
       (net 36 /~CF_DASP))
@@
   )
   (module LEDs:LED_D3.0mm (layer Front)
-    (at 107.95 100.457)
+    (at 110.5 100.4 180)
     (descr "LED, diameter 3.0mm, 2 pins")
     (tags "LED diameter 3.0mm 2 pins")
-    (fp_text reference D1 (at 1.27 -2.96) (layer F.Fab)
+    (fp_text reference D1 (at 1.27 -2.96 180) (layer F.Fab)
       (effects (font (size 1 1) (thickness 0.15)))
     )
-    (fp_text value LED (at 1.27 2.96) (layer F.Fab)
+    (fp_text value LED (at 1.27 2.96 180) (layer F.Fab)
       (effects (font (size 1 1) (thickness 0.15)))
     )
@@
     (fp_arc (start 1.27 0) (end -0.29 -1.235516) (angle 108.8) (layer F.SilkS) (width 0.12))
     (fp_arc (start 1.27 0) (end -0.23 -1.16619) (angle 284.3) (layer F.Fab) (width 0.1))
-    (pad 2 thru_hole circle (at 2.54 0) (size 1.8 1.8) (drill 0.9) (layers *.Cu *.Mask)
+    (pad 2 thru_hole circle (at 2.54 0 180) (size 1.8 1.8) (drill 0.9) (layers *.Cu *.Mask)
       (net 46 "Net-(D1-Pad2)"))
-    (pad 1 thru_hole rect (at 0 0) (size 1.8 1.8) (drill 0.9) (layers *.Cu *.Mask)
+    (pad 1 thru_hole rect (at 0 0 180) (size 1.8 1.8) (drill 0.9) (layers *.Cu *.Mask)
       (net 47 "Net-(D1-Pad1)"))
     (model ${KISYS3DMOD}/LEDs.3dshapes/LED_D3.0mm.wrl
@@
     (descr "3x-dip-switch, Piano, row spacing 7.62 mm (300 mils)")
     (tags "DIP Switch Piano 7.62mm 300mil")
-    (fp_text reference SW3 (at 3.81 -3.17) (layer F.SilkS)
+    (fp_text reference SW3 (at 3.81 -3.17) (layer F.Fab)
       (effects (font (size 1 1) (thickness 0.15)))
     )
@@
     (descr "Through hole angled pin header, 1x02, 2.54mm pitch, 6mm pin length, single row")
     (tags "Through hole angled pin header THT 1x02 2.54mm single row")
-    (fp_text reference P2 (at 4.385 -2.27 90) (layer F.SilkS)
+    (fp_text reference P2 (at 4.385 -2.27 90) (layer F.Fab)
       (effects (font (size 1 1) (thickness 0.15)))
     )
@@
     (fp_line (start 2.2 -2.85) (end -2.21 -2.85) (layer B.CrtYd) (width 0.05))
     (pad 1 smd rect (at -1.5 2 180) (size 0.9 0.9) (layers Back B.Paste B.Mask)
-      (net 47 "Net-(D1-Pad1)"))
+      (net 46 "Net-(D1-Pad2)"))
     (pad 4 smd rect (at -1.5 -2 180) (size 0.9 0.9) (layers Back B.Paste B.Mask))
     (pad 2 smd rect (at -1.5 0.66 180) (size 0.9 0.9) (layers Back B.Paste B.Mask)
@@
       (xy 0.500964 3.601424)) (layer B.SilkS) (width 0.01))
   )
+  (gr_line (start 105.791 88.2) (end 101.981 88.2) (layer B.SilkS) (width 0.1524))
+  (gr_line (start 105.791 97.1) (end 101.981 97.1) (layer B.SilkS) (width 0.1524))
   (gr_line (start 121.796 120.6025) (end 121.796 117.3005) (layer B.SilkS) (width 0.1524))
   (gr_line (start 135.639 117.3005) (end 135.639 124.6665) (layer B.SilkS) (width 0.1524))
@@
   (gr_line (start 182.245 124.587) (end 180.975 123.317) (layer F.SilkS) (width 0.381))
   (gr_line (start 182.245 124.587) (end 166.878 124.587) (layer F.SilkS) (width 0.381))
-  (gr_text + (at 111.8235 87.63) (layer F.SilkS)
+  (gr_text + (at 106.6 87.7) (layer F.SilkS)
     (effects (font (size 1.5 1.5) (thickness 0.3)) (justify mirror))
   )
@@
   (segment (start 173.4927 110.871) (end 173.4927 123.1265) (width 0.2) (layer Back) (net 31))
   (via (at 173.4927 110.871) (size 0.6) (layers Front Back) (net 31))
-  (segment (start 109.4425 103.029) (end 109.5135 103.029) (width 0.2) (layer Back) (net 32) (status 30))
-  (segment (start 109.22 102.8065) (end 109.4425 103.029) (width 0.2) (layer Back) (net 32) (status 30))
-  (segment (start 109.22 99.568) (end 109.22 102.8065) (width 0.2) (layer Back) (net 32) (status 20))
-  (segment (start 165.862 88.011) (end 119.888 88.011) (width 0.2) (layer Back) (net 32) (status 10))
-  (segment (start 117.4611 90.4379) (end 117.4611 92.2794) (width 0.2) (layer Back) (net 32))
+  (segment (start 109.4425 103.029) (end 109.5135 103.029) (width 0.2) (layer Back) (net 32))
+  (segment (start 109.22 102.8065) (end 109.4425 103.029) (width 0.2) (layer Back) (net 32))
+  (segment (start 109.22 99.08) (end 109.22 102.8065) (width 0.2) (layer Back) (net 32))
+  (segment (start 165.862 88.011) (end 119.888 88.011) (width 0.2) (layer Back) (net 32))
   (segment (start 119.888 88.011) (end 117.4611 90.4379) (width 0.2) (layer Back) (net 32))
+  (segment (start 117.4611 90.4379) (end 117.4611 92.2794) (width 0.2) (layer Back) (net 32))
+  (segment (start 110.998 98.7425) (end 109.5575 98.7425) (width 0.2) (layer Back) (net 32))
   (segment (start 117.4611 92.2794) (end 110.998 98.7425) (width 0.2) (layer Back) (net 32))
-  (segment (start 110.998 98.7425) (end 110.0455 98.7425) (width 0.2) (layer Back) (net 32))
-  (segment (start 110.0455 98.7425) (end 109.22 99.568) (width 0.2) (layer Back) (net 32))
+  (segment (start 109.5575 98.7425) (end 109.22 99.08) (width 0.2) (layer Back) (net 32))
   (via (at 141.859 93.853) (size 0.6) (drill 0.3) (layers Front Back) (net 33))
   (segment (start 140.302 93.853) (end 141.859 93.853) (width 0.2) (layer Back) (net 33) (status 10))
@@
   (segment (start 128.652 102.743) (end 126.1745 102.743) (width 0.6) (layer Back) (net 45) (status 10))
   (segment (start 126.1745 102.743) (end 126.111 102.6795) (width 0.6) (layer Back) (net 45))
-  (via (at 144.0815 93.853004) (size 0.6) (drill 0.3) (layers Front Back) (net 46))
-  (segment (start 145.702 93.853) (end 144.081504 93.853) (width 0.2) (layer Back) (net 46) (status 10))
-  (segment (start 144.081504 93.853) (end 144.0815 93.853004) (width 0.2) (layer Back) (net 46))
-  (segment (start 144.653 94.424504) (end 144.0815 93.853004) (width 0.2) (layer Front) (net 46))
-  (segment (start 144.653 96.8375) (end 144.653 94.424504) (width 0.2) (layer Front) (net 46))
-  (segment (start 110.9345 100.457) (end 112.141 99.2505) (width 0.2) (layer Front) (net 46) (status 10))
-  (segment (start 110.49 100.457) (end 110.9345 100.457) (width 0.2) (layer Front) (net 46) (status 30))
-  (segment (start 112.141 99.2505) (end 125.4125 99.2505) (width 0.2) (layer Front) (net 46))
-  (segment (start 125.4125 99.2505) (end 126.492 98.171) (width 0.2) (layer Front) (net 46))
-  (segment (start 126.492 98.171) (end 143.3195 98.171) (width 0.2) (layer Front) (net 46))
-  (segment (start 143.3195 98.171) (end 144.653 96.8375) (width 0.2) (layer Front) (net 46))
-  (segment (start 106.3625 98.8695) (end 107.95 100.457) (width 0.2) (layer Back) (net 47) (status 20))
-  (segment (start 106.3625 96.393) (end 106.3625 98.8695) (width 0.2) (layer Back) (net 47))
-  (segment (start 107.696 95.0595) (end 106.3625 96.393) (width 0.2) (layer Back) (net 47))
-  (segment (start 107.696 92.456) (end 107.696 95.0595) (width 0.2) (layer Back) (net 47))
-  (segment (start 109.5135 90.7735) (end 109.3785 90.7735) (width 0.2) (layer Back) (net 47) (status 30))
-  (segment (start 109.3785 90.7735) (end 107.696 92.456) (width 0.2) (layer Back) (net 47) (status 10))
+  (via (at 144.0815 93.853004) (size 0.6) (drill 0.3) (layers Front Back) (net 47))
+  (segment (start 145.702 93.853) (end 144.081504 93.853) (width 0.2) (layer Back) (net 47) (status 10))
+  (segment (start 144.081504 93.853) (end 144.0815 93.853004) (width 0.2) (layer Back) (net 47))
+  (segment (start 144.653 94.424504) (end 144.0815 93.853004) (width 0.2) (layer Front) (net 47))
+  (segment (start 144.653 96.8375) (end 144.653 94.424504) (width 0.2) (layer Front) (net 47))
+  (segment (start 110.9345 100.457) (end 112.141 99.2505) (width 0.2) (layer Front) (net 47) (status 10))
+  (segment (start 110.49 100.457) (end 110.9345 100.457) (width 0.2) (layer Front) (net 47) (status 30))
+  (segment (start 112.141 99.2505) (end 125.4125 99.2505) (width 0.2) (layer Front) (net 47))
+  (segment (start 125.4125 99.2505) (end 126.492 98.171) (width 0.2) (layer Front) (net 47))
+  (segment (start 126.492 98.171) (end 143.3195 98.171) (width 0.2) (layer Front) (net 47))
+  (segment (start 143.3195 98.171) (end 144.653 96.8375) (width 0.2) (layer Front) (net 47))
+  (segment (start 106.3625 98.8695) (end 107.95 100.457) (width 0.2) (layer Back) (net 46) (status 20))
+  (segment (start 106.3625 96.393) (end 106.3625 98.8695) (width 0.2) (layer Back) (net 46))
+  (segment (start 107.696 95.0595) (end 106.3625 96.393) (width 0.2) (layer Back) (net 46))
+  (segment (start 107.696 92.456) (end 107.696 95.0595) (width 0.2) (layer Back) (net 46))
+  (segment (start 109.5135 90.7735) (end 109.3785 90.7735) (width 0.2) (layer Back) (net 46) (status 30))
+  (segment (start 109.3785 90.7735) (end 107.696 92.456) (width 0.2) (layer Back) (net 46) (status 10))
   (segment (start 126.0475 97.5995) (end 142.4305 97.5995) (width 0.2) (layer Front) (net 48))
   (segment (start 142.4305 97.5995) (end 143.637 96.393) (width 0.2) (layer Front) (net 48))

Commit message: Add files via upload
Parts:
- removed REF***: OSHW-Logo_7.5x8mm_SilkScreen, Symbols:OSHW-Logo_7.5x8mm_SilkScreen
- added G***: LOGO, Custom:Monotech_Logo_150, B.Cu at (215.5, 139.1)
- C1, C2, C3, C4, C5, C6: value 0.1uF -> 100nF; footprint Capacitors_SMD:C_0805_HandSoldering -> Capacitor_SMD:C_0805_2012Metric_Pad1.15x1.40mm_HandSolder
- C7, C8, R1, R2: footprint Capacitors_SMD:C_0805_HandSoldering -> Capacitor_SMD:C_0805_2012Metric_Pad1.15x1.40mm_HandSolder
- D1: value LED -> IDE LED; footprint LEDs:LED_D3.0mm -> LED_THT:LED_D3.0mm
- JP1, JP2, JP3: footprint Custom:SolderJumper-2_P1.3mm_Open_Pad1.0x1.5mm -> Jumper:SolderJumper-2_P1.3mm_Open_Pad1.0x1.5mm
- P1: footprint Custom:CF_Slot_ACON_CFA17_Reverse -> Custom:CF_Slot_3M_N7E50-7516TS0884
- P2: value LED -> IDE LED; footprint Pin_Headers:Pin_Header_Angled_1x02_Pitch2.54mm -> Connector_PinHeader_2.54mm:PinHeader_1x02_P2.54mm_Horizontal
- RN1, RN2, RN3, RN4: footprint Resistors_SMD:R_Array_Convex_4x1206 -> Resistor_SMD:R_Array_Convex_4x1206
- SW3, SW4: footprint Buttons_Switches_THT:SW_DIP_x3_W7.62mm_Piano -> Button_Switch_THT:SW_DIP_SPSTx03_Slide_9.78x9.8mm_W7.62mm_P2.54mm
- U1: footprint Housings_DIP:DIP-28_W15.24mm_Socket -> Package_DIP:DIP-28_W15.24mm_Socket
- U2, U3: footprint Housings_SOIC:SOIC-20W_7.5x12.8mm_Pitch1.27mm -> Package_SO:SOIC-20W_7.5x12.8mm_P1.27mm
- U4, U5: footprint Housings_SOIC:SOIC-14_3.9x8.7mm_Pitch1.27mm -> Package_SO:SOIC-14_3.9x8.7mm_P1.27mm
- moved G*** 84.2 mm to (200.9, 137.3)
- moved P2 80.4 mm to (186.4, 114.8), turned to 180 degrees
- moved SW1 80.2 mm to (179.1, 129.3)
- moved SW2 80.1 mm to (179.1, 120.4)
- moved D1 79.9 mm to (185.8, 127.0)
- moved RN2 79.5 mm to (183.0, 131.3)
- moved RN4 79.0 mm to (183.2, 117.1)
- moved JP3 78.1 mm to (186.7, 131.7)
- moved C2 76.5 mm to (228.5, 132.5)
- moved C4 76.5 mm to (207.3, 128.5)
- moved C8 76.5 mm to (228.5, 134.6)
- moved R2 76.5 mm to (244.7, 136.1)
- moved U1 76.5 mm to (237.1, 115.8)
- moved C1 76.5 mm to (244.7, 128.8)
- moved C5 76.5 mm to (198.8, 132.2)
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Connections:
- net /RESETDRV renamed /RSTDRV
- P1 pad 24: (no net) -> Net-(P1-Pad24)
- P1 pad 25: (no net) -> Net-(P1-Pad25)
- P1 pad 26: (no net) -> Net-(P1-Pad26)
- P1 pad 27: (no net) -> Net-(P1-Pad27)
- P1 pad 28: (no net) -> Net-(P1-Pad28)
- P1 pad 29: (no net) -> Net-(P1-Pad29)
- P1 pad 30: (no net) -> Net-(P1-Pad30)
- P1 pad 31: (no net) -> Net-(P1-Pad31)
- P1 pad 33: (no net) -> Net-(P1-Pad33)
- P1 pad 37: (no net) -> Net-(P1-Pad37)
- P1 pad 40: (no net) -> Net-(P1-Pad40)
- P1 pad 46: (no net) -> Net-(P1-Pad46)
- P1 pad 47: (no net) -> Net-(P1-Pad47)
- P1 pad 48: (no net) -> Net-(P1-Pad48)
- P1 pad 49: (no net) -> Net-(P1-Pad49)
- RN4 pad 4: (no net) -> Net-(RN4-Pad4)
- SW1 pad 3: (no net) -> Net-(SW1-Pad3)
- SW2 pad 1: (no net) -> Net-(SW2-Pad1)
- U1 pad 26: (no net) -> Net-(U1-Pad26)
- U4 pad 11: (no net) -> Net-(U4-Pad11)
- U4 pad 8: (no net) -> Net-(U4-Pad8)
- U5 pad 4: (no net) -> Net-(U5-Pad4)
Routing:
- net /D3: track 95.5 -> 39.2 mm, vias 1 -> 0
- net /D4: track 91.4 -> 53.6 mm, vias 0 -> 1
- net /D2: track 30.5 -> 63.6 mm
- net /AEN: track 94.1 -> 61.4 mm, vias 1 -> 3
- net Net-(RN3-Pad1): track 62.8 -> 92.4 mm
- net /~CF_DASP: track 70.9 -> 41.4 mm, vias 3 -> 1
- net /~MEMW: track 120.2 -> 92.3 mm, vias 0 -> 1
- net /D5: track 84.9 -> 58.7 mm, vias 1 -> 0
- net /D1: track 35.8 -> 60.4 mm
- net /~IOR: track 33.1 -> 9.82 mm
- net /D6: track 81.2 -> 59.1 mm, vias 3 -> 1
- net /~ROM_CS: track 30.5 -> 52.3 mm, vias 1 -> 0
- net /D0: track 39.5 -> 59.3 mm
- net /~IOW: track 32.4 -> 13.8 mm
- net Net-(JP1-Pad2): track 64.7 -> 82.0 mm, vias 2 -> 0
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- added copper zone on F.Cu, net GND
- removed copper zone on F.Cu, net VCC
Other:
- board size 81.3 x 49 mm -> 81.3 x 51.6 mm
- rule pad_to_mask_clearance: 0.254 -> 0
- board text added: "123 111 300 011 320 101 340 001 360 110 380 010 3A0 100 3C0 000 3E0"
- board text added: "Rev 1.1"
- board text removed: "123 111 300 110 320 101 340 100 360 011 380 010 3A0 001 3C0 000 3E0"
- board text removed: "Rev 1"
