File: xt-cf-mini.sch (KiCad schematic (older format))
At the start: 30 parts, among them P1 CF_CARD, P2 LED, SW1 ROM Enable, SW2 ROM Write Enable, SW3 ROM Addr, SW4 IDE Addr, U1 28C64, U2 74LS688, U3 74LS688, U4 74LS32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

Commit message: Add files via upload
Parts:
- BUS1: symbol xt-cf-rescue:BUSPC_DEV -> xt-cf-mini-rescue:BUSPC_DEV-xt-cf-rescue
- C1, C2, C3, C4, C5, C6: symbol xt-cf-rescue:C -> xt-cf-mini-rescue:C-xt-cf-rescue
- C7, C8: symbol xt-cf-rescue:CP1 -> xt-cf-mini-rescue:CP1-xt-cf-rescue
- D1: symbol xt-cf-rescue:LED -> Device:LED
- P1: symbol xt-cf-rescue:CF_CARD -> xt-cf-mini-rescue:CF_CARD-xt-cf-rescue
- P2: symbol xt-cf-rescue:CONN_2 -> xt-cf-mini-rescue:CONN_2-xt-cf-rescue
- R1, R2: symbol xt-cf-rescue:R -> xt-cf-mini-rescue:R-xt-cf-rescue
- U1: symbol xt-cf-rescue:28C64 -> xt-cf-mini-rescue:28C64-xt-cf-rescue
- U2, U3: symbol xt-cf-rescue:74LS688 -> xt-cf-mini-rescue:74LS688-xt-cf-rescue
- U4: symbol xt-cf-rescue:74LS32 -> xt-cf-mini-rescue:74LS32-xt-cf-rescue
- U5: symbol xt-cf-rescue:74LS04 -> xt-cf-mini-rescue:74LS04-xt-cf-rescue
Connections:
- net at U5.10: now also D1.1 (K); no longer D1.2 (K)
- net at RN4.1 (R1.1): now also D1.2 (A); no longer D1.1 (A)
Changed lines of the file:
@@
 Connection ~ 9500 9100
 Wire Wire Line
-	12600 6400 12700 6400
+	12600 6400 12750 6400
 Wire Wire Line
 	10900 5300 10400 5300
@@
 	4250 6000 4250 6900
 $Comp
-L xt-cf-rescue:GND #PWR01
+L xt-cf-mini-rescue:GND-xt-cf-rescue #PWR01
 U 1 1 511C4410
 P 9500 9600
@@
 GND
 $Comp
-L xt-cf-rescue:74LS04 U5
+L xt-cf-mini-rescue:74LS04-xt-cf-rescue U5
 U 2 1 5116DA71
 P 10000 9500
@@
 NoConn ~ 1700 1700
 $Comp
-L xt-cf-rescue:GND #PWR02
+L xt-cf-mini-rescue:GND-xt-cf-rescue #PWR02
 U 1 1 5116EEA5
 P 4700 3550
@@
 $EndComp
 $Comp
-L xt-cf-rescue:R R1
+L xt-cf-mini-rescue:R-xt-cf-rescue R1
 U 1 1 5116ED7F
 P 11150 5300
@@
 $EndComp
 $Comp
-L xt-cf-rescue:GND #PWR04
+L xt-cf-mini-rescue:GND-xt-cf-rescue #PWR04
 U 1 1 5116ED4F
 P 11400 5300
@@
 $EndComp
 $Comp
-L xt-cf-rescue:CONN_2 P2
+L xt-cf-mini-rescue:CONN_2-xt-cf-rescue P2
 U 1 1 5116EC3C
 P 12900 7250
@@
 $EndComp
 $Comp
-L xt-cf-rescue:LED D1
+L Device:LED D1
 U 1 1 5116EC22
 P 12900 6400
@@
 F 3 "" H 12900 6400 50  0001 C CNN
 	1    12900 6400
-	-1   0    0    1
+	1    0    0    -1
 $EndComp
 NoConn ~ 10400 9500
@@
 A4
 $Comp
-L xt-cf-rescue:74LS04 U5
+L xt-cf-mini-rescue:74LS04-xt-cf-rescue U5
 U 1 1 5116DA6E
 P 7300 1600
@@
 A9
 $Comp
-L xt-cf-rescue:74LS04 U5
+L xt-cf-mini-rescue:74LS04-xt-cf-rescue U5
 U 3 1 5116DA77
 P 11200 6000
@@
 $EndComp
 $Comp
-L xt-cf-rescue:74LS04 U5
+L xt-cf-mini-rescue:74LS04-xt-cf-rescue U5
 U 6 1 5116DA69
 P 12200 6800
@@
 $EndComp
 $Comp
-L xt-cf-rescue:74LS04 U5
+L xt-cf-mini-rescue:74LS04-xt-cf-rescue U5
 U 5 1 5116DA67
 P 12200 6400
@@
 $EndComp
 $Comp
-L xt-cf-rescue:74LS04 U5
+L xt-cf-mini-rescue:74LS04-xt-cf-rescue U5
 U 4 1 5116DA62
 P 11200 6400
@@
 $EndComp
 $Comp
-L xt-cf-rescue:74LS32 U4
+L xt-cf-mini-rescue:74LS32-xt-cf-rescue U4
 U 4 1 5116DA5C
 P 10000 9050
@@
 $EndComp
 $Comp
-L xt-cf-rescue:74LS32 U4
+L xt-cf-mini-rescue:74LS32-xt-cf-rescue U4
 U 3 1 5116DA57
 P 10000 8650
@@
 $EndComp
 $Comp
-L xt-cf-rescue:74LS32 U4
+L xt-cf-mini-rescue:74LS32-xt-cf-rescue U4
 U 2 1 5116DA55
 P 8900 1650
@@
 $EndComp
 $Comp
-L xt-cf-rescue:74LS32 U4
+L xt-cf-mini-rescue:74LS32-xt-cf-rescue U4
 U 1 1 5116DA4F
 P 8900 2050
@@
 $EndComp
 $Comp
-L xt-cf-rescue:74LS688 U3
+L xt-cf-mini-rescue:74LS688-xt-cf-rescue U3
 U 1 1 5116DA04
 P 7500 3000
@@
 D0
 $Comp
-L xt-cf-rescue:CF_CARD P1
+L xt-cf-mini-rescue:CF_CARD-xt-cf-rescue P1
 U 1 1 5116D113
 P 11600 3000
@@
 RDY/~BUSY
 $Comp
-L xt-cf-rescue:28C64 U1
+L xt-cf-mini-rescue:28C64-xt-cf-rescue U1
 U 1 1 509149DC
 P 7300 6150
@@
 $EndComp
 $Comp
-L xt-cf-rescue:GND #PWR08
+L xt-cf-mini-rescue:GND-xt-cf-rescue #PWR08
 U 1 1 508E02DD
 P 1300 9400
@@
 $EndComp
 $Comp
-L xt-cf-rescue:BUSPC_DEV BUS1
+L xt-cf-mini-rescue:BUSPC_DEV-xt-cf-rescue BUS1
 U 1 1 508DEF42
 P 2600 2700
@@
 $EndComp
 $Comp
-L xt-cf-rescue:GND #PWR09
+L xt-cf-mini-rescue:GND-xt-cf-rescue #PWR09
 U 1 1 508DF5E3
 P 4250 7000
@@
 $EndComp
 $Comp
-L xt-cf-rescue:GND #PWR011
+L xt-cf-mini-rescue:GND-xt-cf-rescue #PWR011
 U 1 1 508DF511
 P 1550 7100
@@
 A19
 $Comp
-L xt-cf-rescue:74LS688 U2
+L xt-cf-mini-rescue:74LS688-xt-cf-rescue U2
 U 1 1 508DF197
 P 4950 6200
@@
 ~ROM_CS
 $Comp
-L xt-cf-rescue:GND #PWR014
+L xt-cf-mini-rescue:GND-xt-cf-rescue #PWR014
 U 1 1 4EF92A22
 P 1200 2200
@@
 $EndComp
 $Comp
-L xt-cf-rescue:GND #PWR016
+L xt-cf-mini-rescue:GND-xt-cf-rescue #PWR016
 U 1 1 4EF92983
 P 1200 4300
@@
 $EndComp
 $Comp
-L xt-cf-rescue:CP1 C8
+L xt-cf-mini-rescue:CP1-xt-cf-rescue C8
 U 1 1 4EF13BF8
 P 3400 9000
@@
 $EndComp
 $Comp
-L xt-cf-rescue:GND #PWR017
+L xt-cf-mini-rescue:GND-xt-cf-rescue #PWR017
 U 1 1 4ED6C9CC
 P 1200 1300
@@
 Settings
 $Comp
-L xt-cf-rescue:CP1 C7
+L xt-cf-mini-rescue:CP1-xt-cf-rescue C7
 U 1 1 4D4252FF
 P 3100 9000
@@
 $EndComp
 $Comp
-L xt-cf-rescue:C C6
+L xt-cf-mini-rescue:C-xt-cf-rescue C6
 U 1 1 4C69F1EE
 P 2800 9000
@@
 $EndComp
 $Comp
-L xt-cf-rescue:C C1
+L xt-cf-mini-rescue:C-xt-cf-rescue C1
 U 1 1 4C69F1DA
 P 1300 9000
@@
 $EndComp
 $Comp
-L xt-cf-rescue:C C2
+L xt-cf-mini-rescue:C-xt-cf-rescue C2
 U 1 1 4C69F1D9
 P 1600 9000
@@
 $EndComp
 $Comp
-L xt-cf-rescue:C C3
+L xt-cf-mini-rescue:C-xt-cf-rescue C3
 U 1 1 4C69F1D8
 P 1900 9000
@@
 $EndComp
 $Comp
-L xt-cf-rescue:C C4
+L xt-cf-mini-rescue:C-xt-cf-rescue C4
 U 1 1 4C69F1D7
 P 2200 9000
@@
 $EndComp
 $Comp
-L xt-cf-rescue:C C5
+L xt-cf-mini-rescue:C-xt-cf-rescue C5
 U 1 1 4C69F1D6
 P 2500 9000
@@
 $EndComp
 Wire Wire Line
-	13100 6400 13150 6400
+	13050 6400 13150 6400
 Wire Wire Line
 	13150 6400 13150 6250
@@
 	6000 3300 6900 3300
 $Comp
-L xt-cf-rescue:R R2
+L xt-cf-mini-rescue:R-xt-cf-rescue R2
 U 1 1 5BF70D4E
 P 11150 5500
@@
 $EndComp
 $Comp
-L xt-cf-rescue:GND #PWR0101
+L xt-cf-mini-rescue:GND-xt-cf-rescue #PWR0101
 U 1 1 5BF70DB2
 P 11400 5500

Commit message: Add files via upload
Parts:
- C1, C2, C3, C4, C5, C6: value 0.1uF -> 100nF; footprint Capacitors_SMD:C_0805_HandSoldering -> Capacitor_SMD:C_0805_2012Metric_Pad1.15x1.40mm_HandSolder
- C7, C8, R1, R2: footprint Capacitors_SMD:C_0805_HandSoldering -> Capacitor_SMD:C_0805_2012Metric_Pad1.15x1.40mm_HandSolder
- D1: value LED -> IDE LED; footprint LEDs:LED_D3.0mm -> LED_THT:LED_D3.0mm
- JP1, JP2, JP3: footprint Custom:SolderJumper-2_P1.3mm_Open_Pad1.0x1.5mm -> Jumper:SolderJumper-2_P1.3mm_Open_Pad1.0x1.5mm
- P1: footprint Custom:CF_Slot_ACON_CFA17_Reverse -> Custom:CF_Slot_3M_N7E50-7516TS0884
- P2: value LED -> IDE LED; footprint Pin_Headers:Pin_Header_Angled_1x02_Pitch2.54mm -> Connector_PinHeader_2.54mm:PinHeader_1x02_P2.54mm_Horizontal
- RN1, RN2, RN3, RN4: footprint Resistors_SMD:R_Array_Convex_4x1206 -> Resistor_SMD:R_Array_Convex_4x1206
- SW3, SW4: footprint Buttons_Switches_THT:SW_DIP_x3_W7.62mm_Piano -> Button_Switch_THT:SW_DIP_SPSTx03_Slide_9.78x9.8mm_W7.62mm_P2.54mm
- U1: footprint Housings_DIP:DIP-28_W15.24mm_Socket -> Package_DIP:DIP-28_W15.24mm_Socket
- U2, U3: footprint Housings_SOIC:SOIC-20W_7.5x12.8mm_Pitch1.27mm -> Package_SO:SOIC-20W_7.5x12.8mm_P1.27mm
- U4, U5: footprint Housings_SOIC:SOIC-14_3.9x8.7mm_Pitch1.27mm -> Package_SO:SOIC-14_3.9x8.7mm_P1.27mm
Connections:
- net RESETDRV renamed RSTDRV
